File: mm_mcu.kicad_sch (KiCad schematic)
At the start: 18 parts, among them J1 Conn_ARM_JTAG_SWD_10, U1 STM32F030C8Tx

Commit message: tp3
Parts:
- renumbered BOOT0 to BOOT1, C6 to C3, C1 to C4, C2 to C5, C3 to C6, C4 to C7, C5 to C8, J1 to J2, R5 to R10, R1 to R2, R6 to R3, R7 to R4, R8 to R5, R9 to R6, R2 to R7, R3 to R8, R4 to R9, U1 to U2
