File: minimouse.kicad_pcb (KiCad board)
At the start: 2 copper layers, 90 x 85 mm, 22 parts, among them J1 Conn_ARM_JTAG_SWD_10, J5 Conn_01x02, M1 N20_encoder, M2 N20_encoder, U1 STM32F030C8Tx, U4 HC-SR04

Commit message: tp3
Parts:
- added C1: C, Capacitor_SMD:C_0603_1608Metric, F.Cu at (118.9, 44.7)
- added C10: 2.2 uF, Capacitor_SMD:C_0603_1608Metric, F.Cu at (83.5, 30.5)
- added C11: C, Capacitor_SMD:C_0603_1608Metric, F.Cu at (123.5, 30.5)
- added C12: 2.2uF, Capacitor_SMD:C_0603_1608Metric, F.Cu at (78.9, 23.5)
- added C2: C, Capacitor_SMD:C_0603_1608Metric, F.Cu at (118.9, 47.2)
- added C9: 2.2 uF, Capacitor_SMD:C_0603_1608Metric, F.Cu at (94.2, 30.5)
- added Cen1: 10nF, Capacitor_SMD:C_0603_1608Metric, F.Cu at (100.2, 30.5)
- added Croff1: 22nF, Capacitor_SMD:C_0603_1608Metric, F.Cu at (100.2, 33.0)
- added Cs1: 2.2uF, Capacitor_SMD:C_0603_1608Metric, F.Cu at (100.2, 35.5)
- added Cspol1: 22uF, Capacitor_SMD:C_0603_1608Metric, F.Cu at (100.2, 38.0)
- added Csteb1: 1nF, Capacitor_SMD:C_0603_1608Metric, F.Cu at (100.2, 40.5)
- added D1: LED, LED_SMD:LED_0603_1608Metric, F.Cu at (122.9, 49.2)
- added J3: Conn_01x06, Connector_PinHeader_2.54mm:PinHeader_1x06_P2.54mm_Vertical, F.Cu at (89.8, 31.6)
- added J4: Conn_01x06, Connector_PinHeader_2.54mm:PinHeader_1x06_P2.54mm_Vertical, F.Cu at (79.2, 31.6)
- added J5: Conn_01x04, Connector_PinHeader_2.54mm:PinHeader_1x04_P2.54mm_Vertical, F.Cu at (119.2, 31.6)
- added R1: R, Resistor_SMD:R_0603_1608Metric, F.Cu at (118.9, 49.8)
- added R11: 18Kohm, Resistor_SMD:R_0603_1608Metric, F.Cu at (100.2, 43.0)
- added R12: R, Resistor_SMD:R_0603_1608Metric, F.Cu at (104.2, 30.5)
- added R13: R, Resistor_SMD:R_0603_1608Metric, F.Cu at (104.2, 33.0)
- added R14: 100, Resistor_SMD:R_0603_1608Metric, F.Cu at (94.2, 33.0)
- added R15: 100, Resistor_SMD:R_0603_1608Metric, F.Cu at (94.2, 35.5)
- added R16: 100, Resistor_SMD:R_0603_1608Metric, F.Cu at (83.5, 33.0)
- added R17: 100, Resistor_SMD:R_0603_1608Metric, F.Cu at (83.5, 35.5)
- added R18: R, Resistor_SMD:R_0603_1608Metric, F.Cu at (123.5, 33.0)
- added R19: 100, Resistor_SMD:R_0603_1608Metric, F.Cu at (78.9, 26.0)
- added RRroff1: 1kohm, Resistor_SMD:R_0603_1608Metric, F.Cu at (104.2, 35.5)
- added Rcoff1: 1kohm, Resistor_SMD:R_0603_1608Metric, F.Cu at (104.2, 38.0)
- added Ren1: 18kohm, Resistor_SMD:R_0603_1608Metric, F.Cu at (104.2, 40.5)
- added Rrsnsb1: 330mohm, Resistor_SMD:R_2512_6332Metric, F.Cu at (110.5, 31.7)
- added Rsnsa1: 330mohm, Resistor_SMD:R_2512_6332Metric, F.Cu at (110.5, 36.6)
- added U1: LP5907MFX-1.2, Package_TO_SOT_SMD:SOT-23-5, F.Cu at (123.5, 45.7)
- added U3: STSPIN240, Package_DFN_QFN:VQFN-16-1EP_3x3mm_P0.5mm_EP1.8x1.8mm, F.Cu at (108.8, 41.7)
- added U4: HC-SR04, minimouse:HC-SR04, F.Cu at (99.9, 20.9)
- moved C8 62.5 mm to (185.6, 77.1), turned to -90 degrees
- moved C6 37.6 mm to (178.7, 76.4), turned to -90 degrees
- moved C4 33.7 mm to (172.9, 77.1), turned to -90 degrees
- moved C7 31.4 mm to (182.2, 77.1), turned to 90 degrees
- moved C5 30.7 mm to (175.4, 77.9)
- moved C3 27.4 mm to (170.3, 77.1)
- moved R8 17.6 mm to (134.8, 83.9)
- moved R9 9.79 mm to (134.8, 99.2)
- moved J2 9.40 mm to (172.9, 86.0)
- moved R6 3.81 mm to (144.9, 78.0)
- moved U2 3.14 mm to (153.0, 89.5)
- moved R2 2.22 mm to (150.0, 78.9)
- moved R5 2.22 mm to (151.8, 78.9)
- moved R10 2.19 mm to (143.9, 99.2)
- renumbered BOOT0 to BOOT1, C6 to C3, C1 to C4, C2 to C5, C3 to C6, C4 to C7, C5 to C8, J5 to J1, J1 to J2, R5 to R10, R1 to R2, R6 to R3, R7 to R4, R8 to R5, R9 to R6, R2 to R7, R3 to R8, R4 to R9, U1 to U2
Connections:
- C3 pad 2: GND -> +BATT
- C4 pad 2: GND -> +BATT
- C5 pad 2: GND -> +BATT
- C6 pad 2: GND -> +BATT
- C7 pad 2: GND -> +BATT
- C8 pad 2: GND -> +BATT
- J1 pad 1: GND -> +BATT
- J2 pad 3: GND -> +BATT
- J2 pad 5: GND -> +BATT
- J2 pad 9: GND -> +BATT
- R2 pad 2: GND -> +BATT
- R5 pad 1: /mcu/UART1_TX -> /external_uart/EXT_UART_RX
- U2 pad 23: GND -> +BATT
- U2 pad 43: /mcu/UART1_RX -> /external_uart/EXT_UART_TX
- U2 pad 47: GND -> +BATT
- U2 pad 8: GND -> +BATT

Commit message: tp4
Parts:
- moved R14 104.2 mm to (177.9, 94.9), turned to 90 degrees
- moved J3 101.8 mm to (165.2, 100.0), turned to 90 degrees
- moved R15 100.0 mm to (174.6, 94.9), turned to 90 degrees
- moved R19 95.0 mm to (161.9, 72.1)
- moved C12 93.2 mm to (158.4, 72.1)
- moved J4 89.8 mm to (137.3, 100.0), turned to -90 degrees
- moved C10 89.8 mm to (142.4, 98.2), turned to -90 degrees
- moved R16 79.9 mm to (133.9, 94.9), turned to 90 degrees
- moved R17 74.7 mm to (128.9, 94.9), turned to 90 degrees
- moved U4 70.7 mm to (151.3, 69.5)
- moved C11 64.8 mm to (117.0, 94.9)
- moved D1 62.9 mm to (157.6, 101.8), turned to 90 degrees
- moved Croff1 62.7 mm to (120.3, 92.4)
- moved Rrsnsb1 62.1 mm to (137.3, 87.7), turned to 90 degrees
- moved R1 62.1 mm to (157.6, 98.3), turned to 90 degrees
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Routing:
- net Net-(D1-K): track 0.00 -> 23.9 mm
- net Net-(U3-SENSEB): track 0.00 -> 14.9 mm
- net Net-(U3-REF): track 0.00 -> 13.6 mm
- net /motorB/MA: track 0.00 -> 11.5 mm
- net +3.3V: track 0.00 -> 5.92 mm
- net (no net): track 0.00 -> 5.62 mm
- net unconnected-(R12-Pad1): track 0.00 -> 5.11 mm
- net +BATT: track 0.00 -> 4.58 mm
- net Net-(U3-SENSEA): track 0.00 -> 4.55 mm
- net unconnected-(Ren1-Pad2): track 0.00 -> 4.01 mm
