File: mm_motor_control.kicad_sch (KiCad schematic)
At the start: 0 parts

Commit message: fin tp2
Parts:
- added Cen: 10nF, symbol Device:C
- added Croff: 22nF, symbol Device:C
- added Cs: 2.2uF, symbol Device:C
- added Cspol: 22uF, symbol Device:C
- added Csteb: 1nF, symbol Device:C
- added R1: 18Kohm, symbol Device:R
- added R10, R11: R, symbol Device:R
- added RRroff, Rcoff: 1kohm, symbol Device:R
- added Ren: 18kohm, symbol Device:R
- added Rrsnsb, Rsnsa: 330mohm, symbol Device:R
- added U3: STSPIN240, Package_DFN_QFN:VQFN-16-1EP_3x3mm_P0.5mm_EP1.8x1.8mm, symbol Driver_Motor:STSPIN240
Connections:
- net OUT_A1: now also U3.3 (OUTA1)
- net OUT_A2: now also U3.5 (OUTA2)
- net OUT_B1: now also U3.10 (OUTB1)
- net OUT_B2: now also U3.8 (OUTB2)
- net PHASE_A: now also U3.1 (PHA)
- net PHASE_B: now also U3.15 (PHB)
- net PWM_A: now also U3.2 (PWMA)
- net PWM_B: now also U3.16 (PWMB)
- new net: Csteb.1, R1.2, U3.14 (STBY/RESET)
- new net: Cs.1, Cspol.1, U3.6 (VS)
- new net: Cen.1, Ren.1, U3.13 (EN/FLT)
- new net: RRroff.1, Rcoff.1, U3.12 (TOFF)
- new net: R10.1, R11.2, U3.11 (REF)
- new net: Rrsnsb.1, U3.9 (SENSEB)
- new net: Croff.1, Rcoff.2
- new net: Rsnsa.1, U3.4 (SENSEA)
- new net +3.3V: R1.1
- new net GND: Cen.2, Croff.2, Cs.2, Cspol.2, Csteb.2, R10.2, RRroff.2, Rrsnsb.2, Rsnsa.2, U3.7 (GND)

Commit message: tp3
Parts:
- Cen1: renamed from Cen; footprint (none) -> Capacitor_SMD:C_0603_1608Metric
- Croff1: renamed from Croff; footprint (none) -> Capacitor_SMD:C_0603_1608Metric
- Cs1: renamed from Cs; footprint (none) -> Capacitor_SMD:C_0603_1608Metric
- Cspol1: renamed from Cspol; footprint (none) -> Capacitor_SMD:C_0603_1608Metric
- Csteb1: renamed from Csteb; footprint (none) -> Capacitor_SMD:C_0603_1608Metric
- R11: renamed from R1; footprint (none) -> Resistor_SMD:R_0603_1608Metric
- R12: renamed from R11; footprint (none) -> Resistor_SMD:R_0603_1608Metric
- R13: renamed from R10; footprint (none) -> Resistor_SMD:R_0603_1608Metric
- RRroff1: renamed from RRroff; footprint (none) -> Resistor_SMD:R_0603_1608Metric
- Rcoff1: renamed from Rcoff; footprint (none) -> Resistor_SMD:R_0603_1608Metric
- Ren1: renamed from Ren; footprint (none) -> Resistor_SMD:R_0603_1608Metric
- Rrsnsb1: renamed from Rrsnsb; footprint (none) -> Resistor_SMD:R_2512_6332Metric
- Rsnsa1: renamed from Rsnsa; footprint (none) -> Resistor_SMD:R_2512_6332Metric

Commit message: tp4
Other:
- moved on the sheet: Cen1, Croff1, Cs1, Cspol1, Csteb1, R11, R13, RRroff1, Rcoff1, Ren1, Rrsnsb1, Rsnsa1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
